File: eagle files/SSM4.brd (EAGLE design)
At the start: 62.2 x 51.7 mm, 12 parts

Commit message: Add files via upload
Routing:
- net MCN: track 38.4 -> 42.9 mm
- net VCC: track 100.3 -> 96.9 mm
- net VCC_IN: track 43.2 -> 40.1 mm
- net STEP_UP_ENABLE: track 49.9 -> 47.1 mm, vias 0 -> 1
- net D7: track 31.4 -> 33.4 mm
- net MCP: track 47.1 -> 45.3 mm
- net BATT+: track 29.9 -> 28.7 mm
- net D2: track 43.4 -> 42.2 mm
